File: HDMI_INPUT.sch (KiCad schematic (older format))
At the start: 52 parts, among them J1 HDMI_A, U1 TPD4S010DQAR, U2 TPD4S010DQAR, U3 ABM3B-24.000MHZ-B2-T, U4 TPS2061, U5 ADV7611

Commit message: Added pdata lines and ran bus connections
Parts:
- C1, C10, C11, C12, C15, C16, C17, C18, C19, C2, C20, C21, C22, C23, C24, C25, C26, C27, C28, C3, C4, C5, C6, C7, C8, C9, R10: footprint (none) -> Capacitors_SMD:C_0402
- FB1, FB2, FB3, FB4, FB5: footprint (none) -> Capacitors_SMD:C_0603
- J1: footprint ADV7611:LQFP-64_TH_10x10mm_Pitch0.5mm -> hdmi:FCI_10029449-11[13]RLF
- R1, R2, R3, R4, R5, R6, R7, R8, R9: footprint (none) -> Resistors_SMD:R_0402
- RP1, RP2, RP3: footprint (none) -> rpack:RPACK-8_0616
- U5: footprint MODULE -> ADV7611:LQFP-64_TH_10x10mm_Pitch0.5mm
Connections:
- net labels added: PDATA[0..23]
- net labels removed: PDATA
