File: $MSP430.sch (KiCad schematic (older format))
At the start: 23 parts, among them P1 CONN_02X07, SW1 2M1-SP1-T2-B4-M6RE, U6 MSP430F2274TRHAR

Commit message: Started PCB Layout, added mounting holes, connectors, in correct locations
Parts:
- H1, H2, H3: renamed from H?; footprint (none) -> Mounting_Holes:MountingHole_4.3mm_M4_Pad_Via
Connections:
- wire segments 104 -> 81
Changed lines of the file:
@@
 $EndComp
 Wire Wire Line
-	4350 2750 4750 2750
-Wire Wire Line
-	4750 2750 6750 2750
+	4350 2750 6750 2750
 Wire Wire Line
 	4750 2750 4750 2650
@@
 	8500 2250 8800 2250
 Wire Wire Line
-	8800 2050 8800 2250
-Wire Wire Line
-	8800 2250 8800 2350
+	8800 2050 8800 2350
 Wire Wire Line
 	8800 2350 8500 2350
@@
 TEST
 Wire Wire Line
-	8350 6350 9550 6350
-Wire Wire Line
-	9550 6350 9700 6350
-Wire Wire Line
-	8350 6450 9400 6450
-Wire Wire Line
-	9400 6450 9700 6450
+	8350 6350 9700 6350
+Wire Wire Line
+	8350 6450 9700 6450
 $Comp
 L R R20
@@
 	9400 5800 9550 5800
 Wire Wire Line
-	9550 5650 9550 5800
-Wire Wire Line
-	9550 5800 9550 5900
+	9550 5650 9550 5900
 Connection ~ 9550 5800
 Wire Wire Line
@@
 $EndComp
 Wire Wire Line
-	8500 7350 8500 7450
-Wire Wire Line
-	8500 7450 8500 7550
-Wire Wire Line
-	8500 7550 8500 7650
-Wire Wire Line
-	8500 7650 8500 7800
+	8500 7350 8500 7800
 Wire Wire Line
 	8500 7350 8350 7350
@@
 	1100 1200 1400 1200
 Wire Wire Line
-	1700 1200 1850 1200
-Wire Wire Line
-	1850 1200 2150 1200
-Wire Wire Line
-	2150 1200 2450 1200
-Wire Wire Line
-	2450 1200 3250 1200
+	1700 1200 3250 1200
 Wire Wire Line
 	2450 1200 2450 1300
@@
 $EndComp
 Wire Wire Line
-	2450 1600 2450 1700
-Wire Wire Line
-	2450 1700 2450 1750
-Wire Wire Line
-	1850 1700 2150 1700
-Wire Wire Line
-	2150 1700 2450 1700
+	2450 1600 2450 1750
+Wire Wire Line
+	1850 1700 2450 1700
 Connection ~ 2450 1700
 Wire Wire Line
@@
 MSP_VDD3V3
 Wire Wire Line
-	8350 3700 8500 3700
-Wire Wire Line
-	8500 3700 9250 3700
+	8350 3700 9250 3700
 Wire Wire Line
 	8350 3800 8500 3800
 Wire Wire Line
-	8500 3700 8500 3800
-Wire Wire Line
-	8500 3800 8500 3900
+	8500 3700 8500 3900
 Connection ~ 8500 3700
 Wire Wire Line
@@
 MSP_VDD3V3
 Wire Wire Line
-	9150 4300 9450 4300
-Wire Wire Line
-	9450 4300 9750 4300
-Wire Wire Line
-	9750 4300 10050 4300
-Wire Wire Line
-	10050 4300 10350 4300
-Wire Wire Line
-	10350 4300 11050 4300
+	9150 4300 11050 4300
 Wire Wire Line
 	9150 4300 9150 4400
@@
 $EndComp
 Wire Wire Line
-	3000 7400 3250 7400
-Wire Wire Line
-	3250 7400 3700 7400
+	3000 7400 3700 7400
 Wire Wire Line
 	3250 7400 3250 7550
@@
 POWER_ON
 $Comp
-L HOLE1 H?
+L HOLE1 H1
 U 1 1 56F98079
 P 12650 1000
-F 0 "H?" H 12650 1150 60  0000 C CNN
+F 0 "H1" H 12650 1150 60  0000 C CNN
 F 1 "HOLE1" H 12650 850 60  0000 C CNN
-F 2 "" H 12650 1000 60  0000 C CNN
+F 2 "Mounting_Holes:MountingHole_4.3mm_M4_Pad_Via" H 12650 1000 60  0001 C CNN
 F 3 "" H 12650 1000 60  0000 C CNN
 	1    12650 1000
@@
 $EndComp
 $Comp
-L HOLE1 H?
+L HOLE1 H2
 U 1 1 56F9810C
 P 12650 1400
-F 0 "H?" H 12650 1550 60  0000 C CNN
+F 0 "H2" H 12650 1550 60  0000 C CNN
 F 1 "HOLE1" H 12650 1250 60  0000 C CNN
-F 2 "" H 12650 1400 60  0000 C CNN
+F 2 "Mounting_Holes:MountingHole_4.3mm_M4_Pad_Via" H 12650 1400 60  0001 C CNN
 F 3 "" H 12650 1400 60  0000 C CNN
 	1    12650 1400
@@
 $EndComp
 $Comp
-L HOLE1 H?
+L HOLE1 H3
 U 1 1 56F9815A
 P 12650 1800
-F 0 "H?" H 12650 1950 60  0000 C CNN
+F 0 "H3" H 12650 1950 60  0000 C CNN
 F 1 "HOLE1" H 12650 1650 60  0000 C CNN
-F 2 "" H 12650 1800 60  0000 C CNN
+F 2 "Mounting_Holes:MountingHole_4.3mm_M4_Pad_Via" H 12650 1800 60  0001 C CNN
 F 3 "" H 12650 1800 60  0000 C CNN
 	1    12650 1800
@@
 	12850 1000 12950 1000
 Wire Wire Line
-	12950 1000 12950 1400
-Wire Wire Line
-	12950 1400 12950 1800
-Wire Wire Line
-	12950 1800 12950 1800
+	12950 1000 12950 1950
 Wire Wire Line
 	12950 1800 12850 1800
@@
 Connection ~ 12950 1400
 $Comp
-L GND #PWR?
+L GND #PWR049
 U 1 1 56F98389
 P 12950 1950
-F 0 "#PWR?" H 12950 1700 50  0001 C CNN
+F 0 "#PWR049" H 12950 1700 50  0001 C CNN
 F 1 "GND" H 12950 1800 50  0000 C CNN
 F 2 "" H 12950 1950 60  0000 C CNN
@@
 	1    0    0    -1
 $EndComp
-Wire Wire Line
-	12950 1950 12950 1800
 Connection ~ 12950 1800
 $EndSCHEMATC
