File: HDMI2RGB.kicad_pcb (KiCad board)
At the start: 4 copper layers, 58.4 x 63.5 mm, 106 parts, among them J1 HDMI_A, J2 QTH-030-02-L-DA, J3 RAPC712x, P1 CONN_02X07, SW1 2M1-SP1-T2-B4-M6RE, U1 TPD4S010DQAR, U10 TPS62260, U11 TPS62260, U2 TPD4S010DQAR, U3 ABM3B-24.000MHZ-B2-T, U4 TPS2061, U5 ADV7611, U6 MSP430F2274TRHAR, U7 SN74AUP1G06DCKR, U8 SN74AUP1G07DCKR, U9 SN74AUP1G06DCKR

Commit message: First Final -- Waiting for Checker
Parts:
- added D5: LED, Capacitors_SMD:C_0603, F.Cu at (101.6, 107.2)
- added D6: LED, Capacitors_SMD:C_0603, F.Cu at (101.6, 102.1)
- added P2: CONN_01X06, Pin_Headers:Pin_Header_Straight_1x06, F.Cu at (78.2, 125.3)
- added P3: CONN_01X06, Pin_Headers:Pin_Header_Straight_1x06, F.Cu at (77.9, 77.1)
- added R31: 270, Resistors_SMD:R_0402, F.Cu at (101.6, 109.9)
- added R34: 270, Resistors_SMD:R_0402, F.Cu at (101.6, 104.8)
- added U12: SN74AUP1G06DCKR, TO_SOT_Packages_SMD:SC-70-5, F.Cu at (98.6, 109.2)
- added U13: SN74AUP1G06DCKR, TO_SOT_Packages_SMD:SC-70-5, F.Cu at (98.6, 104.1)
- moved R17 41.9 mm to (78.3, 79.2), turned to 180 degrees
- moved R19 41.5 mm to (77.9, 80.7), turned to 180 degrees
- moved R22 37.4 mm to (73.3, 81.3)
- moved R21 37.0 mm to (73.2, 79.9)
- moved R23 35.0 mm to (70.7, 79.9)
- moved C32 21.0 mm to (90.0, 80.8), turned to 90 degrees
- moved R12 19.7 mm to (88.4, 80.8), turned to 270 degrees
- moved R13 19.1 mm to (91.6, 80.9), turned to 90 degrees
- moved R24 15.3 mm to (101.6, 125.1)
- moved U7 15.3 mm to (98.6, 124.5)
- moved C33 15.2 mm to (98.6, 122.4)
- moved R14 13.9 mm to (70.2, 92.3), turned to 90 degrees
- moved D4 12.8 mm to (92.7, 65.7), turned to 90 degrees
- moved D3 12.7 mm to (101.6, 112.3), turned to 270 degrees
- moved R15 10.5 mm to (65.8, 90.8), turned to 180 degrees
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Connections:
- U6 pad 12: Net-(U6-Pad12) -> PROJ_ON
- U6 pad 15: /MSP430/PB_UP -> /MSP430/DEBUG1
- U6 pad 16: /MSP430/PB_DOWN -> /MSP430/DEBUG2
- U6 pad 17: /MSP430/PB_LEFT -> /MSP430/POWER_ON
- U6 pad 18: /MSP430/PB_RIGHT -> /MSP430/PB_UP
- U6 pad 19: /MSP430/PB_SELECT -> /MSP430/PB_DOWN
- U6 pad 20: Net-(U6-Pad20) -> /MSP430/PB_LEFT
- U6 pad 21: Net-(U6-Pad21) -> /MSP430/PB_RIGHT
- U6 pad 22: Net-(U6-Pad22) -> /MSP430/PB_SELECT
- U6 pad 9: Net-(U6-Pad9) -> HOST_IRQ
Routing:
- net GND: track 27.2 -> 274.9 mm, vias 10 -> 21
- net +3V3: track 97.9 -> 187.7 mm, vias 4 -> 6
- net +1V8: track 6.59 -> 67.8 mm, vias 0 -> 2
- net HOST_IRQ: track 0.00 -> 49.9 mm, vias 0 -> 4
- net SYSPWR: track 58.3 -> 105.4 mm, vias 4 -> 6
- net PROJ_ON: track 0.00 -> 36.6 mm, vias 0 -> 2
- net /MSP430/DEBUG1: track 0.00 -> 32.9 mm
- net /HDMI_INPUT/ADV_VDD1V8: track 42.0 -> 74.4 mm, vias 2 -> 3
- net /MSP430/TEST: track 0.00 -> 31.8 mm
- net /MSP430/MSP_VDD3V3: track 39.9 -> 70.0 mm, vias 4 -> 7
- net RESET: track 0.00 -> 29.3 mm, vias 0 -> 1
- net SPI0_CLK: track 0.00 -> 28.7 mm
- net /MSP430/DEBUG2: track 0.00 -> 28.4 mm
- net SPI0_CSZ0: track 0.00 -> 25.6 mm, vias 0 -> 1
- net /MSP430/POWER_ON: track 0.00 -> 24.3 mm
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Other:
- rule trace_min: 0.1524 -> 0.006
- rule via_min_size: 0.5588 -> 0.022
